File: heardware/kicad-project/USB-Screen.sch (KiCad schematic (older format))
At the start: 22 parts, among them J1 USB_B_Micro, J2 Conn_01x04, J3 USB_C_Receptacle_USB2.0, K1 SW_4*4mm, K2 SW_4*4mm, K3 SW_4*4mm, Q1 NPN, U1 ZJY154T-PG04, U2 CH551, U3 SC662

Commit message: 添加俩个3D封装
Parts:
- J1: symbol Connector:USB_B_Micro -> USB-Screen-rescue:USB_B_Micro-Connector
- J3: footprint Connector_USB:USB_C_Receptacle_Palconn_UTC16-G -> Connector_USB:USB_C_Receptacle_Steady_UTC16-G
- K1: footprint USB-Screen:SW_4mm_4mm -> Button_Switch_SMD:SW_Push_1P1T_NO_4x4mm_H2.0mm; symbol USB_Screen_Library:SW_4*4mm -> Switch:SW_Push
- K2: renamed from K3; footprint USB-Screen:SW_4mm_4mm -> Button_Switch_SMD:SW_Push_1P1T_NO_4x4mm_H2.0mm; symbol USB_Screen_Library:SW_4*4mm -> Switch:SW_Push
- K3: renamed from K2; footprint USB-Screen:SW_4mm_4mm -> Button_Switch_SMD:SW_Push_1P1T_NO_4x4mm_H2.0mm; symbol USB_Screen_Library:SW_4*4mm -> Switch:SW_Push
Connections:
- net GND: now also K1.2, K2.2, K3.2; no longer K1.3, K1.4, K2.3, K2.4, K3.3, K3.4
- net K1: no longer K1.2
- net K2: now also K2.1, U2.9 (P1.1); no longer K3.1, K3.2, U2.10 (P3.3)
- net K3: now also K3.1, U2.10 (P3.3); no longer K2.1, K2.2, U2.9 (P1.1)
Changed lines of the file:
@@
 $EndComp
 $Comp
-L Connector:USB_B_Micro J1
+L USB-Screen-rescue:USB_B_Micro-Connector J1
 U 1 1 5F605CF0
 P 3600 1850
@@
 	6100 4150 5700 4150
 Wire Wire Line
+	6100 4350 5700 4350
+Wire Wire Line
 	6100 4250 5700 4250
-Wire Wire Line
-	6100 4350 5700 4350
 Text Label 6100 4150 2    50   ~ 0
 PWM
@@
 	4400 4250 4600 4250
 Wire Wire Line
-	4400 4350 4600 4350
+	4600 4350 4400 4350
 Text Label 4400 3650 0    50   ~ 0
 RST
 Text Label 4400 4250 0    50   ~ 0
 DC
-Text Label 4400 4350 0    50   ~ 0
+Text Label 4600 4350 2    50   ~ 0
 K1
+Text Label 6100 4350 2    50   ~ 0
+K2
 Text Label 6100 4250 2    50   ~ 0
-K2
-Text Label 6100 4350 2    50   ~ 0
 K3
 NoConn ~ 3900 2050
@@
 F 0 "J3" H 1857 2667 50  0000 C CNN
 F 1 "USB_C_Receptacle_USB2.0" H 1857 2576 50  0000 C CNN
-F 2 "Connector_USB:USB_C_Receptacle_Palconn_UTC16-G" H 1900 1800 50  0001 C CNN
+F 2 "Connector_USB:USB_C_Receptacle_Steady_UTC16-G" H 1900 1800 50  0001 C CNN
 F 3 "https://www.usb.org/sites/default/files/documents/usb_type-c.zip" H 1900 1800 50  0001 C CNN
 	1    1750 1800
@@
 L power:GND #PWR05
 U 1 1 5F892224
-P 7800 4000
-F 0 "#PWR05" H 7800 3750 50  0001 C CNN
-F 1 "GND" H 7805 3827 50  0000 C CNN
-F 2 "" H 7800 4000 50  0001 C CNN
-F 3 "" H 7800 4000 50  0001 C CNN
-	1    7800 4000
-	1    0    0    -1
-$EndComp
-$Comp
-L USB_Screen_Library:SW_4*4mm K1
+P 9400 3500
+F 0 "#PWR05" H 9400 3250 50  0001 C CNN
+F 1 "GND" H 9405 3327 50  0000 C CNN
+F 2 "" H 9400 3500 50  0001 C CNN
+F 3 "" H 9400 3500 50  0001 C CNN
+	1    9400 3500
+	1    0    0    -1
+$EndComp
+$Comp
+L Switch:SW_Push K1
 U 1 1 5F8A4CE4
-P 7700 4100
-F 0 "K1" H 7700 4575 50  0000 C CNN
-F 1 "SW_4*4mm" H 7700 4484 50  0000 C CNN
-F 2 "USB-Screen:SW_4mm_4mm" H 7700 4100 50  0001 C CNN
-F 3 "" H 7700 4100 50  0001 C CNN
-	1    7700 4100
+P 7750 3500
+F 0 "K1" H 7750 3750 50  0000 C CNN
+F 1 "SW_4*4mm" H 7750 3650 50  0000 C BNN
+F 2 "Button_Switch_SMD:SW_Push_1P1T_NO_4x4mm_H2.0mm" H 7750 3500 50  0001 C CNN
+F 3 "" H 7750 3500 50  0001 C CNN
+	1    7750 3500
 	1    0    0    -1
 $EndComp
@@
 L power:GND #PWR0113
 U 1 1 5F8A68B9
-P 7600 4000
-F 0 "#PWR0113" H 7600 3750 50  0001 C CNN
-F 1 "GND" H 7605 3827 50  0000 C CNN
-F 2 "" H 7600 4000 50  0001 C CNN
-F 3 "" H 7600 4000 50  0001 C CNN
-	1    7600 4000
-	1    0    0    -1
-$EndComp
-Text Label 7900 3850 2    50   ~ 0
+P 7950 3500
+F 0 "#PWR0113" H 7950 3250 50  0001 C CNN
+F 1 "GND" H 7955 3327 50  0000 C CNN
+F 2 "" H 7950 3500 50  0001 C CNN
+F 3 "" H 7950 3500 50  0001 C CNN
+	1    7950 3500
+	1    0    0    -1
+$EndComp
+Text Label 7450 3500 0    50   ~ 0
 K1
 Wire Wire Line
-	7800 3850 7900 3850
-Text Label 7500 3850 0    50   ~ 0
-K1
-Wire Wire Line
-	7500 3850 7600 3850
-$Comp
-L power:GND #PWR0115
-U 1 1 5F8BAA20
-P 8350 4000
-F 0 "#PWR0115" H 8350 3750 50  0001 C CNN
-F 1 "GND" H 8355 3827 50  0000 C CNN
-F 2 "" H 8350 4000 50  0001 C CNN
-F 3 "" H 8350 4000 50  0001 C CNN
-	1    8350 4000
-	1    0    0    -1
-$EndComp
-$Comp
-L USB_Screen_Library:SW_4*4mm K2
+	7450 3500 7550 3500
+$Comp
+L Switch:SW_Push K3
 U 1 1 5F8BAA26
-P 8250 4100
-F 0 "K2" H 8250 4575 50  0000 C CNN
-F 1 "SW_4*4mm" H 8250 4484 50  0000 C CNN
-F 2 "USB-Screen:SW_4mm_4mm" H 8250 4100 50  0001 C CNN
-F 3 "" H 8250 4100 50  0001 C CNN
-	1    8250 4100
-	1    0    0    -1
-$EndComp
-$Comp
-L power:GND #PWR0116
-U 1 1 5F8BAA2C
-P 8150 4000
-F 0 "#PWR0116" H 8150 3750 50  0001 C CNN
-F 1 "GND" H 8155 3827 50  0000 C CNN
-F 2 "" H 8150 4000 50  0001 C CNN
-F 3 "" H 8150 4000 50  0001 C CNN
-	1    8150 4000
-	1    0    0    -1
-$EndComp
-Text Label 8450 3850 2    50   ~ 0
-K2
-Wire Wire Line
-	8350 3850 8450 3850
-Text Label 8050 3850 0    50   ~ 0
-K2
-Wire Wire Line
-	8050 3850 8150 3850
-$Comp
-L power:GND #PWR0117
-U 1 1 5F8BD0BF
-P 8900 4000
-F 0 "#PWR0117" H 8900 3750 50  0001 C CNN
-F 1 "GND" H 8905 3827 50  0000 C CNN
-F 2 "" H 8900 4000 50  0001 C CNN
-F 3 "" H 8900 4000 50  0001 C CNN
-	1    8900 4000
-	1    0    0    -1
-$EndComp
-$Comp
-L USB_Screen_Library:SW_4*4mm K3
+P 9200 3500
+F 0 "K3" H 9200 3750 50  0000 C CNN
+F 1 "SW_4*4mm" H 9200 3650 50  0000 C CNN
+F 2 "Button_Switch_SMD:SW_Push_1P1T_NO_4x4mm_H2.0mm" H 9200 3500 50  0001 C CNN
+F 3 "" H 9200 3500 50  0001 C CNN
+	1    9200 3500
+	1    0    0    -1
+$EndComp
+$Comp
+L Switch:SW_Push K2
 U 1 1 5F8BD0C5
-P 8800 4100
-F 0 "K3" H 8800 4575 50  0000 C CNN
-F 1 "SW_4*4mm" H 8800 4484 50  0000 C CNN
-F 2 "USB-Screen:SW_4mm_4mm" H 8800 4100 50  0001 C CNN
-F 3 "" H 8800 4100 50  0001 C CNN
-	1    8800 4100
+P 8500 3500
+F 0 "K2" H 8500 3750 50  0000 C CNN
+F 1 "SW_4*4mm" H 8500 3650 50  0000 C CNN
+F 2 "Button_Switch_SMD:SW_Push_1P1T_NO_4x4mm_H2.0mm" H 8500 3500 50  0001 C CNN
+F 3 "" H 8500 3500 50  0001 C CNN
+	1    8500 3500
 	1    0    0    -1
 $EndComp
@@
 L power:GND #PWR0118
 U 1 1 5F8BD0CB
-P 8700 4000
-F 0 "#PWR0118" H 8700 3750 50  0001 C CNN
-F 1 "GND" H 8705 3827 50  0000 C CNN
-F 2 "" H 8700 4000 50  0001 C CNN
-F 3 "" H 8700 4000 50  0001 C CNN
-	1    8700 4000
-	1    0    0    -1
-$EndComp
-Text Label 9000 3850 2    50   ~ 0
+P 8700 3500
+F 0 "#PWR0118" H 8700 3250 50  0001 C CNN
+F 1 "GND" H 8705 3327 50  0000 C CNN
+F 2 "" H 8700 3500 50  0001 C CNN
+F 3 "" H 8700 3500 50  0001 C CNN
+	1    8700 3500
+	1    0    0    -1
+$EndComp
+Wire Wire Line
+	8900 3500 9000 3500
+Text Label 8900 3500 0    50   ~ 0
 K3
 Wire Wire Line
-	8900 3850 9000 3850
-Text Label 8600 3850 0    50   ~ 0
-K3
-Wire Wire Line
-	8600 3850 8700 3850
+	8200 3500 8300 3500
+Text Label 8200 3500 0    50   ~ 0
+K2
 $EndSCHEMATC
